File: RasPi-BplusHAT.sch (EAGLE design)
At the start: 7 parts, among them K1 PIN20X2, U1 EEPROM24

Commit message: delete cruft
Parts:
- removed C1: 100nF, resistor:C-EUC0805K
- removed CFG: (no value), FLYFISH:PIN2_100
- removed R1, R2: 3k9, resistor:R-EU_M0805
- removed R3: 1k, resistor:R-EU_M0805
- removed U1: EEPROM24, FLYFISH:EEPROM24
Connections:
- removed net N$1: K1.28, R1.1, U1.SCL
- removed net N$2: K1.27, R2.1, U1.SDA
- removed net N$3: CFG.1, R3.1, U1.WP
- net +3V3: no longer C1.1, R1.2, R2.2, R3.2, U1.VCC
- net GND: no longer C1.2, CFG.2, U1.A0, U1.A1, U1.A2, U1.GND
Other:
- note removed: "FLYFISH TECHNOLOGIES d.o.o."
- note removed: "Ivan Zilic"
- note removed: "v0.1"
Changed lines of the file:
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@@
 <part name="K1" library="FLYFISH" deviceset="PIN20X2" device=""/>
 <part name="FRAME1" library="frames" deviceset="A3L-LOC" device=""/>
-<part name="U1" library="FLYFISH" deviceset="EEPROM24" device=""/>
 <part name="GND10" library="supply1" deviceset="GND" device=""/>
-<part name="R1" library="resistor" deviceset="R-EU_" device="M0805" value="3k9">
-<attribute name="TOLERANCE" value="5%"/>
-</part>
-<part name="+3V10" library="supply1" deviceset="+3V3" device=""/>
-<part name="GND1" library="supply1" deviceset="GND" device=""/>
 <part name="+3V1" library="supply1" deviceset="+3V3" device=""/>
-<part name="C1" library="resistor" deviceset="C-EU" device="C0805K" value="100nF">
-<attribute name="DIELECTRIC" value="X7R"/>
-</part>
-<part name="R2" library="resistor" deviceset="R-EU_" device="M0805" value="3k9">
-<attribute name="TOLERANCE" value="5%"/>
-</part>
-<part name="R3" library="resistor" deviceset="R-EU_" device="M0805" value="1k">
-<attribute name="TOLERANCE" value="5%"/>
-</part>
-<part name="CFG" library="FLYFISH" deviceset="PIN2" device="_100"/>
-<part name="+3V4" library="supply1" deviceset="+3V3" device=""/>
-<part name="+3V5" library="supply1" deviceset="+3V3" device=""/>
-<part name="GND2" library="supply1" deviceset="GND" device=""/>
 <part name="GND3" library="supply1" deviceset="GND" device=""/>
 <part name="P+1" library="supply1" deviceset="+5V" device=""/>
@@
 <text x="289.56" y="20.32" size="1.778" layer="94" ratio="15">Drawn by:</text>
 <text x="289.56" y="16.51" size="1.778" layer="94" ratio="15">Checked  by:</text>
-<text x="289.56" y="5.08" size="1.778" layer="94">FLYFISH TECHNOLOGIES d.o.o.</text>
-<text x="309.88" y="20.32" size="1.778" layer="94">Ivan Zilic</text>
-<text x="374.65" y="5.08" size="2.54" layer="94" ratio="10">v0.1</text>
 </plain>
 <instances>
 <instance part="K1" gate="G$1" x="50.8" y="152.4" rot="R180"/>
 <instance part="FRAME1" gate="G$1" x="0" y="0"/>
-<instance part="U1" gate="G$1" x="50.8" y="215.9" smashed="yes">
-<attribute name="NAME" x="48.26" y="224.79" size="1.778" layer="95"/>
-<attribute name="VALUE" x="43.18" y="205.74" size="1.778" layer="96"/>
-</instance>
 <instance part="GND10" gate="1" x="60.96" y="121.92"/>
-<instance part="R1" gate="G$1" x="68.58" y="223.52" smashed="yes" rot="R90">
-<attribute name="TOLERANCE" x="68.58" y="223.52" size="1.778" layer="96" rot="R90" display="off"/>
-<attribute name="NAME" x="71.12" y="223.7486" size="1.778" layer="95"/>
-<attribute name="VALUE" x="71.12" y="221.488" size="1.778" layer="96"/>
-</instance>
-<instance part="+3V10" gate="G$1" x="63.5" y="238.76" smashed="yes">
-<attribute name="VALUE" x="66.04" y="241.3" size="1.778" layer="96" rot="R180"/>
-</instance>
-<instance part="GND1" gate="1" x="38.1" y="205.74"/>
 <instance part="+3V1" gate="G$1" x="38.1" y="182.88" smashed="yes">
 <attribute name="VALUE" x="40.64" y="185.42" size="1.778" layer="96" rot="R180"/>
 </instance>
-<instance part="C1" gate="G$1" x="20.32" y="215.9">
-<attribute name="DIELECTRIC" x="20.32" y="215.9" size="1.778" layer="96" display="off"/>
-</instance>
-<instance part="R2" gate="G$1" x="78.74" y="223.52" smashed="yes" rot="R90">
-<attribute name="TOLERANCE" x="78.74" y="223.52" size="1.778" layer="96" rot="R90" display="off"/>
-<attribute name="NAME" x="81.28" y="223.7486" size="1.778" layer="95"/>
-<attribute name="VALUE" x="81.28" y="221.488" size="1.778" layer="96"/>
-</instance>
-<instance part="R3" gate="G$1" x="38.1" y="228.6" smashed="yes" rot="R90">
-<attribute name="TOLERANCE" x="38.1" y="228.6" size="1.778" layer="96" rot="R90" display="off"/>
-<attribute name="NAME" x="40.64" y="228.8286" size="1.778" layer="95"/>
-<attribute name="VALUE" x="40.64" y="226.568" size="1.778" layer="96"/>
-</instance>
-<instance part="CFG" gate="G$1" x="33.02" y="220.98" smashed="yes">
-<attribute name="NAME" x="29.21" y="223.52" size="1.778" layer="95"/>
-<attribute name="VALUE" x="29.21" y="214.63" size="1.778" layer="96"/>
-</instance>
-<instance part="+3V4" gate="G$1" x="38.1" y="238.76" smashed="yes">
-<attribute name="VALUE" x="40.64" y="241.3" size="1.778" layer="96" rot="R180"/>
-</instance>
-<instance part="+3V5" gate="G$1" x="20.32" y="223.52" smashed="yes">
-<attribute name="VALUE" x="22.86" y="226.06" size="1.778" layer="96" rot="R180"/>
-</instance>
-<instance part="GND2" gate="1" x="20.32" y="205.74"/>
 <instance part="GND3" gate="1" x="40.64" y="121.92"/>
 <instance part="P+1" gate="1" x="60.96" y="182.88" smashed="yes">
@@
 <nets>
 <net name="GND" class="0">
-<segment>
-<pinref part="U1" gate="G$1" pin="A2"/>
-<pinref part="GND1" gate="1" pin="GND"/>
-<wire x1="40.64" y1="218.44" x2="38.1" y2="218.44" width="0.1524" layer="91"/>
-<wire x1="38.1" y1="218.44" x2="38.1" y2="215.9" width="0.1524" layer="91"/>
-<pinref part="U1" gate="G$1" pin="GND"/>
-<wire x1="38.1" y1="215.9" x2="38.1" y2="213.36" width="0.1524" layer="91"/>
-<wire x1="38.1" y1="213.36" x2="38.1" y2="210.82" width="0.1524" layer="91"/>
-<wire x1="38.1" y1="210.82" x2="38.1" y2="208.28" width="0.1524" layer="91"/>
-<wire x1="40.64" y1="210.82" x2="38.1" y2="210.82" width="0.1524" layer="91"/>
-<pinref part="U1" gate="G$1" pin="A0"/>
-<wire x1="40.64" y1="213.36" x2="38.1" y2="213.36" width="0.1524" layer="91"/>
-<pinref part="U1" gate="G$1" pin="A1"/>
-<wire x1="40.64" y1="215.9" x2="38.1" y2="215.9" width="0.1524" layer="91"/>
-<junction x="38.1" y="210.82"/>
-<junction x="38.1" y="213.36"/>
-<junction x="38.1" y="215.9"/>
-<pinref part="CFG" gate="G$1" pin="2"/>
-<wire x1="33.02" y1="218.44" x2="38.1" y2="218.44" width="0.1524" layer="91"/>
-<junction x="38.1" y="218.44"/>
-</segment>
-<segment>
-<pinref part="C1" gate="G$1" pin="2"/>
-<pinref part="GND2" gate="1" pin="GND"/>
-<wire x1="20.32" y1="210.82" x2="20.32" y2="208.28" width="0.1524" layer="91"/>
-</segment>
 <segment>
 <pinref part="K1" gate="G$1" pin="9"/>
@@
 <net name="+3V3" class="0">
 <segment>
-<pinref part="U1" gate="G$1" pin="VCC"/>
-<pinref part="+3V10" gate="G$1" pin="+3V3"/>
-<wire x1="60.96" y1="220.98" x2="63.5" y2="220.98" width="0.1524" layer="91"/>
-<wire x1="63.5" y1="220.98" x2="63.5" y2="231.14" width="0.1524" layer="91"/>
-<pinref part="R2" gate="G$1" pin="2"/>
-<wire x1="63.5" y1="231.14" x2="63.5" y2="236.22" width="0.1524" layer="91"/>
-<wire x1="78.74" y1="228.6" x2="78.74" y2="231.14" width="0.1524" layer="91"/>
-<wire x1="78.74" y1="231.14" x2="68.58" y2="231.14" width="0.1524" layer="91"/>
-<pinref part="R1" gate="G$1" pin="2"/>
-<wire x1="68.58" y1="231.14" x2="63.5" y2="231.14" width="0.1524" layer="91"/>
-<wire x1="68.58" y1="228.6" x2="68.58" y2="231.14" width="0.1524" layer="91"/>
-<junction x="63.5" y="231.14"/>
-<junction x="68.58" y="231.14"/>
-</segment>
-<segment>
-<pinref part="R3" gate="G$1" pin="2"/>
-<pinref part="+3V4" gate="G$1" pin="+3V3"/>
-<wire x1="38.1" y1="236.22" x2="38.1" y2="233.68" width="0.1524" layer="91"/>
-</segment>
-<segment>
-<pinref part="C1" gate="G$1" pin="1"/>
-<pinref part="+3V5" gate="G$1" pin="+3V3"/>
-<wire x1="20.32" y1="220.98" x2="20.32" y2="218.44" width="0.1524" layer="91"/>
-</segment>
-<segment>
 <pinref part="K1" gate="G$1" pin="1"/>
 <pinref part="+3V1" gate="G$1" pin="+3V3"/>
@@
 </segment>
 </net>
-<net name="N$1" class="0">
-<segment>
-<pinref part="U1" gate="G$1" pin="SCL"/>
-<pinref part="R1" gate="G$1" pin="1"/>
-<wire x1="60.96" y1="215.9" x2="68.58" y2="215.9" width="0.1524" layer="91"/>
-<wire x1="68.58" y1="215.9" x2="68.58" y2="218.44" width="0.1524" layer="91"/>
-<pinref part="K1" gate="G$1" pin="28"/>
-<wire x1="58.42" y1="142.24" x2="68.58" y2="142.24" width="0.1524" layer="91"/>
-<wire x1="68.58" y1="142.24" x2="68.58" y2="215.9" width="0.1524" layer="91"/>
-<junction x="68.58" y="215.9"/>
-</segment>
-</net>
-<net name="N$2" class="0">
-<segment>
-<pinref part="U1" gate="G$1" pin="SDA"/>
-<pinref part="R2" gate="G$1" pin="1"/>
-<wire x1="60.96" y1="213.36" x2="78.74" y2="213.36" width="0.1524" layer="91"/>
-<wire x1="78.74" y1="213.36" x2="78.74" y2="218.44" width="0.1524" layer="91"/>
-<pinref part="K1" gate="G$1" pin="27"/>
-<wire x1="43.18" y1="142.24" x2="30.48" y2="142.24" width="0.1524" layer="91"/>
-<wire x1="30.48" y1="142.24" x2="30.48" y2="111.76" width="0.1524" layer="91"/>
-<wire x1="30.48" y1="111.76" x2="78.74" y2="111.76" width="0.1524" layer="91"/>
-<wire x1="78.74" y1="111.76" x2="78.74" y2="213.36" width="0.1524" layer="91"/>
-<junction x="78.74" y="213.36"/>
-</segment>
-</net>
-<net name="N$3" class="0">
-<segment>
-<pinref part="U1" gate="G$1" pin="WP"/>
-<pinref part="R3" gate="G$1" pin="1"/>
-<wire x1="40.64" y1="220.98" x2="38.1" y2="220.98" width="0.1524" layer="91"/>
-<wire x1="38.1" y1="220.98" x2="38.1" y2="223.52" width="0.1524" layer="91"/>
-<pinref part="CFG" gate="G$1" pin="1"/>
-<wire x1="33.02" y1="220.98" x2="38.1" y2="220.98" width="0.1524" layer="91"/>
-<junction x="38.1" y="220.98"/>
-</segment>
-</net>
